File: tof-sensor-board.kicad_pcb (KiCad board)
At the start: 2 copper layers, 22.8 x 16.8 mm, 31 parts, among them U1 STM32F302K8U6, U2 LTC2875, U3 MCP1703, U4 VL53L0X, X1 16MHz

Commit message: Review changes
changes from Rouven's review:
- fix silkscreen too close to pad
- increase CAN and 5V trace width
- make LEDs common VCC
- route voltage regulator 5V input through cpacitor
- add debug connector label
Parts:
- C5: value 22uF -> 10uF
- CONN1: moved to F.Cu
- D2, D3: footprint LEDs:LED-0603 -> Resistors_SMD:R_0603
- moved D2 0.10 mm to (49.2, 54.3), turned to 90 degrees
- moved D3 0.10 mm to (50.8, 54.3), turned to 90 degrees
- turned R6 to 270 degrees
- turned R7 to 270 degrees
Connections:
- D2 pad 1: GND -> Net-(D2-Pad1)
- D2 pad 2: Net-(D2-Pad2) -> VCC
- D3 pad 1: GND -> Net-(D3-Pad1)
- D3 pad 2: Net-(D3-Pad2) -> VCC
- R6 pad 1: Net-(D2-Pad2) -> /Proximity
- R6 pad 2: /Proximity -> Net-(D2-Pad1)
- R7 pad 1: Net-(D3-Pad2) -> /Error
- R7 pad 2: /Error -> Net-(D3-Pad1)
Routing:
- net GND: track 80.9 -> 75.5 mm
- net Net-(CONN2-Pad3): track 27.5 -> 29.9 mm
- net Net-(D2-Pad2): track 1.68 -> 0.00 mm, vias 1 -> 0
- net Net-(D2-Pad1): track 0.00 -> 1.52 mm, vias 0 -> 1
- net Net-(D3-Pad1): track 0.00 -> 1.29 mm, vias 0 -> 1
- net Net-(D3-Pad2): track 1.20 -> 0.00 mm, vias 1 -> 0
- net +5V: track 26.9 -> 27.7 mm
Other:
- board text added: "debug"
