File: tof-sensor-board.sch (KiCad schematic (older format))
At the start: 30 parts, among them U1 STM32F302K8U6, U2 LTC2875, U3 MCP1703, U4 VL53L0X, X1 16MHz

Commit message: routing finished
Connections:
- net Error: now also U1.11 (PA4); no longer U1.12 (PA5)
- net GND: now also MEC1.1, MEC2.1, U1.33 (GND_PAD), U2.9 (GND_PAD)
- net Proximity: now also U1.10 (PA3); no longer U1.11 (PA4)
- no-connect marks 12 -> 10
Other:
- moved on the sheet: MEC2

Commit message: Review changes
changes from Rouven's review:
- fix silkscreen too close to pad
- increase CAN and 5V trace width
- make LEDs common VCC
- route voltage regulator 5V input through cpacitor
- add debug connector label
Parts:
- C5: value 22uF -> 10uF
- D2, D3: footprint LEDs:LED-0603 -> Resistors_SMD:R_0603
Connections:
- net Error: now also R7.1; no longer R7.2
- net GND: no longer D2.1 (K), D3.1 (K)
- net Proximity: now also R6.1; no longer R6.2
- net VCC: now also D2.2 (A), D3.2 (A)
- new net: D2.1 (K), R6.2
- new net: D3.1 (K), R7.2
Other:
- moved on the sheet: D2, D3, R6, R7
Changed lines of the file:
@@
 L LED D2
 U 1 1 55808402
-P 7100 3900
-F 0 "D2" H 7100 4000 50  0000 C CNN
-F 1 "PROXIMITY" H 7100 3800 50  0000 C CNN
-F 2 "LEDs:LED-0603" H 7100 3900 60  0001 C CNN
-F 3 "" H 7100 3900 60  0000 C CNN
-	1    7100 3900
+P 6700 3900
+F 0 "D2" H 6700 4000 50  0000 C CNN
+F 1 "PROXIMITY" H 6700 3800 50  0000 C CNN
+F 2 "Resistors_SMD:R_0603" H 6700 3900 60  0001 C CNN
+F 3 "" H 6700 3900 60  0000 C CNN
+	1    6700 3900
 	-1   0    0    1
 $EndComp
@@
 L LED D3
 U 1 1 55808536
-P 7100 4200
-F 0 "D3" H 7100 4300 50  0000 C CNN
-F 1 "ERROR" H 7100 4100 50  0000 C CNN
-F 2 "LEDs:LED-0603" H 7100 4200 60  0001 C CNN
-F 3 "" H 7100 4200 60  0000 C CNN
-	1    7100 4200
+P 6700 4200
+F 0 "D3" H 6700 4300 50  0000 C CNN
+F 1 "ERROR" H 6700 4100 50  0000 C CNN
+F 2 "Resistors_SMD:R_0603" H 6700 4200 60  0001 C CNN
+F 3 "" H 6700 4200 60  0000 C CNN
+	1    6700 4200
 	-1   0    0    1
 $EndComp
@@
 L R R6
 U 1 1 5580AA34
-P 6650 3900
-F 0 "R6" V 6730 3900 50  0000 C CNN
-F 1 "1k" V 6650 3900 50  0000 C CNN
-F 2 "Resistors_SMD:R_0402" V 6580 3900 30  0001 C CNN
-F 3 "" H 6650 3900 30  0000 C CNN
-	1    6650 3900
+P 7150 3900
+F 0 "R6" V 7230 3900 50  0000 C CNN
+F 1 "1k" V 7150 3900 50  0000 C CNN
+F 2 "Resistors_SMD:R_0402" V 7080 3900 30  0001 C CNN
+F 3 "" H 7150 3900 30  0000 C CNN
+	1    7150 3900
 	0    1    1    0
 $EndComp
@@
 L R R7
 U 1 1 5580AA87
-P 6650 4200
-F 0 "R7" V 6730 4200 50  0000 C CNN
-F 1 "1k" V 6650 4200 50  0000 C CNN
-F 2 "Resistors_SMD:R_0402" V 6580 4200 30  0001 C CNN
-F 3 "" H 6650 4200 30  0000 C CNN
-	1    6650 4200
+P 7150 4200
+F 0 "R7" V 7230 4200 50  0000 C CNN
+F 1 "1k" V 7150 4200 50  0000 C CNN
+F 2 "Resistors_SMD:R_0402" V 7080 4200 30  0001 C CNN
+F 3 "" H 7150 4200 30  0000 C CNN
+	1    7150 4200
 	0    1    1    0
 $EndComp
-$Comp
-L GND #PWR05
-U 1 1 5580AB19
-P 7500 3900
-F 0 "#PWR05" H 7500 3650 50  0001 C CNN
-F 1 "GND" H 7500 3750 50  0000 C CNN
-F 2 "" H 7500 3900 60  0000 C CNN
-F 3 "" H 7500 3900 60  0000 C CNN
-	1    7500 3900
-	1    0    0    -1
-$EndComp
-$Comp
-L GND #PWR06
-U 1 1 5580AB60
-P 7500 4200
-F 0 "#PWR06" H 7500 3950 50  0001 C CNN
-F 1 "GND" H 7500 4050 50  0000 C CNN
-F 2 "" H 7500 4200 60  0000 C CNN
-F 3 "" H 7500 4200 60  0000 C CNN
-	1    7500 4200
-	1    0    0    -1
-$EndComp
-Text Label 6400 3900 2    39   ~ 0
+Text Label 7600 3900 2    39   ~ 0
 Proximity
-Text Label 6400 4200 2    39   ~ 0
+Text Label 7600 4200 2    39   ~ 0
 Error
 Text Label 4600 2300 2    39   ~ 0
@@
 P 9400 5550
 F 0 "C5" H 9425 5650 50  0000 L CNN
-F 1 "22uF" H 9425 5450 50  0000 L CNN
+F 1 "10uF" H 9425 5450 50  0000 L CNN
 F 2 "Capacitors_SMD:C_0603" H 9438 5400 50  0001 C CNN
 F 3 "" H 9400 5550 50  0000 C CNN
@@
 NoConn ~ 4200 2600
 $Comp
-L GND #PWR?
+L GND #PWR023
 U 1 1 57C6DB91
 P 1550 7200
-F 0 "#PWR?" H 1550 6950 50  0001 C CNN
+F 0 "#PWR023" H 1550 6950 50  0001 C CNN
 F 1 "GND" H 1550 7050 50  0000 C CNN
 F 2 "" H 1550 7200 50  0000 C CNN
@@
 $EndComp
 $Comp
-L GND #PWR?
+L GND #PWR024
 U 1 1 57C6DE2C
 P 900 7200
-F 0 "#PWR?" H 900 6950 50  0001 C CNN
+F 0 "#PWR024" H 900 6950 50  0001 C CNN
 F 1 "GND" H 900 7050 50  0000 C CNN
 F 2 "" H 900 7200 50  0000 C CNN
@@
 $EndComp
 $Comp
-L GND #PWR?
+L GND #PWR025
 U 1 1 57C76282
 P 8350 2650
-F 0 "#PWR?" H 8350 2400 50  0001 C CNN
+F 0 "#PWR025" H 8350 2400 50  0001 C CNN
 F 1 "GND" H 8350 2500 50  0000 C CNN
 F 2 "" H 8350 2650 50  0000 C CNN
@@
 Connection ~ 4750 5050
 Wire Wire Line
-	7500 4200 7300 4200
-Wire Wire Line
-	7300 3900 7500 3900
-Wire Wire Line
-	6800 3900 6900 3900
-Wire Wire Line
-	6800 4200 6900 4200
+	7000 4200 6900 4200
+Wire Wire Line
+	6900 3900 7000 3900
 Wire Wire Line
 	6400 3900 6500 3900
@@
 	2600 3350 2700 3350
 $Comp
-L GND #PWR?
+L GND #PWR026
 U 1 1 57C7738E
 P 2600 3350
-F 0 "#PWR?" H 2600 3100 50  0001 C CNN
+F 0 "#PWR026" H 2600 3100 50  0001 C CNN
 F 1 "GND" H 2600 3200 50  0000 C CNN
 F 2 "" H 2600 3350 50  0000 C CNN
@@
 	1    0    0    -1
 $EndComp
+$Comp
+L VCC #PWR?
+U 1 1 57CED075
+P 6400 3900
+F 0 "#PWR?" H 6400 3750 50  0001 C CNN
+F 1 "VCC" H 6400 4050 50  0000 C CNN
+F 2 "" H 6400 3900 50  0000 C CNN
+F 3 "" H 6400 3900 50  0000 C CNN
+	1    6400 3900
+	1    0    0    -1
+$EndComp
+$Comp
+L VCC #PWR?
+U 1 1 57CED0E1
+P 6400 4200
+F 0 "#PWR?" H 6400 4050 50  0001 C CNN
+F 1 "VCC" H 6400 4350 50  0000 C CNN
+F 2 "" H 6400 4200 50  0000 C CNN
+F 3 "" H 6400 4200 50  0000 C CNN
+	1    6400 4200
+	1    0    0    -1
+$EndComp
+Wire Wire Line
+	7300 3900 7600 3900
+Wire Wire Line
+	7600 4200 7300 4200
 $EndSCHEMATC
